Commit message: Clean up unused moveit packages and add planning scene
- Remove *_moveit packages for unused robot variants (cr10af, cr12, cr16,
  cr20, cr20af, cr30h, cr3, cr3af, cr5, cr5af, cr7, me6, nova2, nova2s, nova5)
- Add dobot_planning_scene package (obstacles config, add_scene node)
- Add support.STL meshes for cr10 and disable base_link/support_link collision
- Update cr10 urdf and dobot_moveit launch files

Co-Authored-By: Claude Fable 5 <noreply@anthropic.com>

File: dobot_rviz/urdf/cr10_robot.urdf (robot description, URDF)
Before this commit: robot cr10_robot, 8 links, 7 joints
Links:
- added link support_link, mass 75.163; collision mesh filename=package://dobot_rviz/meshes/cr10/support.STL; visual mesh filename=package://dobot_rviz/meshes/cr10/support.STL
Joints:
- added joint base_support: type fixed, parent base_link, child support_link, origin xyz=0 0 -0.48 rpy=0 0 0
