Commit message: update ompl planner config and joint limit

File: dobot_rviz/urdf/cr10_robot.urdf (robot description, URDF)
Before this commit: robot cr10_robot, 9 links, 8 joints
Joints:
- joint joint1: limit lower=-6.27 upper=6.27 effort=100 velocity=3.14 -> lower=-3.14 upper=3.14 effort=100 velocity=3.14
- joint joint2: limit lower=-6.27 upper=6.27 effort=100 velocity=3.14 -> lower=-3.14 upper=3.14 effort=100 velocity=3.14
- joint joint4: limit lower=-6.27 upper=6.27 effort=100 velocity=3.89 -> lower=-3.14 upper=3.14 effort=100 velocity=3.89
- joint joint5: limit lower=-6.27 upper=6.27 effort=100 velocity=3.89 -> lower=-3.14 upper=3.14 effort=100 velocity=3.89
- joint joint6: limit lower=-6.27 upper=6.27 effort=100 velocity=3.89 -> lower=-3.14 upper=3.14 effort=100 velocity=3.89
